File: voice.sch (KiCad schematic (older format))
At the start: 222 parts

Commit message: added envelope sub sheet
Connections:
- net ENV_2: now reaches R?.2
Other:
- note added: "56K - 100K"
Changed lines of the file:
@@
 LIBS:contrib
 LIBS:valves
+LIBS:MySynthParts
 LIBS:voice-cache
 EELAYER 25 0
@@
 $Descr A1 33110 23386
 encoding utf-8
-Sheet 1 1
+Sheet 1 2
 Title ""
 Date ""
@@
 	1    0    0    -1
 $EndComp
+Text GLabel 29975 20500 2    60   Input ~ 0
+ENV_2
+Wire Wire Line
+	29850 20500 29975 20500
+Text Notes 29525 20725 0    60   ~ 0
+56K - 100K
+$Sheet
+S 23625 8425 2050 1700
+U 57F5D1D5
+F0 "Envelopes" 60
+F1 "envelopes.sch" 60
+$EndSheet
 $EndSCHEMATC

Commit message: ENV1 inverter circuitry captured and simulated.
Parts:
- added Q?: MMBT3904, SOT-23, symbol MMBT3904
- added Q? (x2): MMBT3906, SOT-23, symbol MMBT3906
- added R?: 22K, MyModules:SM0603-R-JRL, symbol R_US
- added R? (x4): 470, MyModules:SM0603-R-JRL, symbol R_US
- added R? (x2): 12K, MyModules:SM0603-R-JRL, symbol R_US
- added R?: 100K, MyModules:SM0603-R-JRL, symbol R_US
- added R?: 180K, MyModules:SM0603-R-JRL, symbol R_US
- added R?: 56K, MyModules:SM0603-R-JRL, symbol R_US
- added U? (x2): LM13700, symbol LM13700
Connections:
- net +12V: now also R?.2, R?.2
- net ENV_2: now also R?.2
- net GND: now also Q?.1 (B), Q?.1 (B), R?.1, R?.1, R?.1, R?.1, R?.1
- new net: Q?.3 (C), U?.1 (x2)
- new net: R?.1, U?.2 (x2)
- new net: R?.2, U?.3 (+) (x2)
- new net: R?.2, U?.4 (-) (x2)
- new net: R?.2, U?.5, U?.5
- new net: Q?.2 (E), R?.1 (x2)
- new net VCF_ENV_MOD: R?.2
Other:
- note added: "18K-28K\n"
- note added: "SIMULATE VCF CONTROL"

Commit message: vcf cutoff control captured
Parts:
- added R? (x3): 68K, MyModules:SM0603-R-JRL, symbol R_US
- added R?: 470K, MyModules:SM0603-R-JRL, symbol R_US
- added R?: 43K, MyModules:SM0603-R-JRL, symbol R_US
- added R? (x3): 100K, MyModules:SM0603-R-JRL, symbol R_US
- added TP?: TEST_POINT, symbol TEST_POINT
- added U? (x3): TL072-, MyModules:TSSOP8-JRL, symbol TL072-
- R?: value 56K -> 27K
Connections:
- net ENV_2: no longer R?.2
- net GND: now also R?.1, U?.3 (+)
- net VCF_CTRL: now also R?.2; no longer Q?.5 (B2), R?.1
- net at R?.2, U?.5, U?.5: now also R?.1, R?.1, R?.1, U?.2 (-)
- net at R?.2: now also R?.2, U?.3 (+)
- net at R?.2, U?.4 (-): now also R?.2
- new net: R?.1, R?.2, U?.1 (x2)
- new net: Q?.5 (B2), R?.1, R?.2, TP?.1
- new net: R?.1, R?.2, U?.2 (-)
- new net KCV_1: R?.1
- new net VCF_KF: R?.2
- new net VCF_TUNE: R?.2
- new net VCO1_RANGE: R?.1
Other:
- note added: "22K - 32K\n"
- note added: "39K - 49K\n"
- note added: "VCF\nCONTROL"
- moved on the sheet: C?, Q?, R?, U?A, U?B

Commit message: pwm circuit added
Parts:
- removed C?: 100p, MyModules:SM0603-C-JRL, symbol C_US
- removed R?: 91K, MyModules:SM0603-R-JRL, symbol R_US
- removed R?: 470K, MyModules:SM0603-R-JRL, symbol R_US
- removed U?: TL072-, MyModules:TSSOP8-JRL, symbol TL072-
- added C?: 100p, MyModules:SM0603-C-JRL, symbol C_US
- added C? (x2): 0.01μ, symbol C_US
- added Q?: MMBT3906, SOT-23, symbol MMBT3906
- added R? (x12): 100K, MyModules:SM0603-R-JRL, symbol R_US
- added R? (x2): 2.2K, MyModules:SM0603-R-JRL, symbol R_US
- added R?: 91K, MyModules:SM0603-R-JRL, symbol R_US
- added R?: 27K, MyModules:SM0603-R-JRL, symbol R_US
- added R?: 68K, MyModules:SM0603-R-JRL, symbol R_US
- added R? (x2): 330, MyModules:SM0603-R-JRL, symbol R_US
- added R?: 12K, MyModules:SM0603-R-JRL, symbol R_US
- added R? (x2): 470K, MyModules:SM0603-R-JRL, symbol R_US
- added R?: 47K, MyModules:SM0603-R-JRL, symbol R_US
- added R? (x2): 10K, MyModules:SM0603-R-JRL, symbol R_US
- added R? (x7): 22K, MyModules:SM0603-R-JRL, symbol R_US
- added R?: 15k, MyModules:SM0603-R-JRL, symbol R_US
- added R? (x2): 18K, MyModules:SM0603-R-JRL, symbol R_US
- added R?: 33K, MyModules:SM0603-R-JRL, symbol R_US
- added R?: 15K, MyModules:SM0603-R-JRL, symbol R_US
- added R?: 30K, MyModules:SM0603-R-JRL, symbol R_US
- added TP?: TEST_POINT, symbol TEST_POINT
- added U? (x2): TL072-, MyModules:TSSOP8-JRL, symbol TL072-
- added U? (x6): CD4053, symbol CD4053
- added U?: LM13700, symbol LM13700
- added U?: RC4558, MyModules:TSSOP8-JRL, symbol TL072-
- added U? (x2): CD4052, symbol CD4052
- added VR? (x2): 20K, symbol POT_US
Connections:
- net VCO1_PITCH_CV is gone; now on net VCO1_XMOD: C?.2, U?.2 (-)
- net XMOD_LEVEL is gone; now on net PWM: R?.1
- net +12V: now also R?.2, R?.2, R?.2, U?.16 (VDD), U?.16 (VDD), U?.16 (Vdd), U?.16 (Vdd), U?.8 (V+), U?.8 (V+)
- net -12V: now also R?.1, R?.1, U?.4 (V-), U?.4 (V-)
- net -5V: now also U?.7 (Vee), U?.8 (VSS), U?.8 (Vss)
- net GND: now also Q?.1 (B), R?.1, R?.1, R?.1, R?.1, R?.1, R?.1, R?.1, U?.1 (Y1), U?.13 (Y1), U?.3 (+), U?.3 (+), U?.3 (+), U?.6 (INH), U?.6 (INH), U?.6 (Inh), U?.6 (Inh), U?.7 (VEE), U?.7 (VEE), U?.7 (Vee), U?.8 (VSS), U?.8 (Vss)
- net KCV_1: now also R?.1
- net PWM: now also C?.2, R?.2, U?.1
- net VCO1_TUNE: now also R?.2
- net VCO1_XMOD: now also R?.1, R?.2, R?.2, R?.2, VR?.2, VR?.3; no longer U?.5
- net at R?.1: now also C?.1, R?.2, U?.1
- net PULSE renamed VCO1_PUSLE
- net VCO1_PUSLE: no longer D?.1 (K), R?.2
- net SAW renamed VCO1_SAW
- net VCO1_SAW: now also U?.5 (Y1); no longer R?.2
- net SINE renamed VCO2_SINE
- net VCO2_SINE: now also U?.1 (Y0)
- net SQUARE renamed VCO1_SQUARE
- net TRIANGLE renamed VCO1_TRI
- net VCO1_TRI: now also U?.1 (Y0)
- net VCF_CTRL renamed VCF_CUTOFF
- net VCO1_IN renamed VCO1
- net VCO1: now also U?.3 (Y)
- net VCO1_SCALE: no longer names the net of R?.1
- net VCO1_SCALE: now also VR?.1
- net VCO2_IN renamed VCO2
- net VCO2: now also U?.3 (Y)
- net XMOD_SOURCE: no longer names the net of R?.1
- net XMOD_SOURCE: now also U?.4 (Z)
- new net: C?.1, R?.1, R?.2, U?.2 (-), U?.5
- new net: R?.1, R?.2, R?.2 (x2)
- new net: C?.2, R?.1, R?.2, R?.2, R?.2, U?.2 (-), VR?.2, VR?.3
- new net: R?.1, VR?.1
- new net: R?.2, U?.2 (Y0)
- new net: Q?.3 (C), U?.1
- new net: R?.1, U?.2
- new net: R?.2, R?.2, U?.3 (+)
- new net: R?.1, R?.2, U?.4 (-)
- new net: C?.1, R?.1, R?.1, R?.2, U?.2 (-), U?.5
- new net: Q?.2 (E), R?.2
- new net: C?.2, R?.1, R?.2, R?.2, TP?.1, U?.1
- new net: R?.1, U?.12 (Y0)
- new net: R?.1, U?.10 (A) (x2)
- new net: R?.1, U?.9 (B) (x2)
- new net: R?.2, U?.11 (S)
- new net: R?.1, R?.2, U?.12 (Y0)
- new net: R?.1, R?.2, U?.13 (Y1)
- new net: U?.14 (Z), U?.3 (Y1)
- new net: R?.1, R?.2, U?.5 (Y0)
- new net: R?.2, U?.9 (S)
- new net ENV_1: R?.1, R?.2
- new net KCV_2: R?.1
- new net LFO: R?.1
- new net NOISE: U?.4 (Y3)
- new net PW/PWM: R?.1
- new net PWM_SEL: R?.1
- new net VCO1_MOD: R?.1, U?.15 (Z)
- new net VCO1_MOD_SW: U?.10 (S)
- new net VCO1_PULSE: U?.2 (Y2)
- new net VCO1_SQARE: U?.4 (Y3)
- new net VCO1_WF-0: R?.2
- new net VCO1_WF-1: R?.2
- new net VCO2_MOD: R?.1, U?.14 (Z)
- new net VCO2_MOD_SW: U?.11 (S)
- new net VCO2_PULSE: D?.1 (K), R?.2, U?.2 (Y2)
- new net VCO2_SAW: R?.2, U?.5 (Y1)
- new net VCO2_TUNE: R?.2
- new net VCO2_WF-0: R?.2
- new net VCO2_WF-1: R?.2
- new net VCO_ENV_MOD: R?.1
- new net VCO_ENV_MOD_BAL: R?.2
- new net VCO_LFO_MOD: R?.1
- new net VCO_MOD_BAL: R?.2
- no-connect marks 1 -> 19
Other:
- note added: "(180K)\n"
- note added: "+10V reference\nin JP8\n"
- note added: "No reference voltage \nhere. May need to adjust R"
- note added: "These are separate ICs\non JP8 module board.\nBecause of cross talk?"
- note added: "VCF CUTOFF is the sum of\nCUTOFF, LFO, VCF PEDAL\nand VCF MOD"
- note added: "ideally replace pot \nwith fixed resistor"
- note added: "low offset LM13700:\nincrease input level, \nreduce Iabc relative \nto BA662 configuration"
- note added: "set initial pitch"
- note removed: "DAC calibration CV here\ninstead of trimmer"
- note removed: "Make this single BJTs\nin case source of C1815 and A1015s\ncan be found?"
- moved on the sheet: C?, D?, Q?, Q?A, Q?B, R?, TC?, U?A, U?B

Commit message: put oscillators into subsheet. slogging through ENV1/ENV2 switching
Parts:
- removed C? (x2): 1n, symbol C_US
- removed C? (x4): 100p, MyModules:SM0603-C-JRL, symbol C_US
- removed C? (x4): 100p, symbol C_US
- removed C? (x2): 10n, symbol C_US
- removed C?: 33p, symbol C_US
- removed D? (x11): 1N4148, symbol D
- removed D?: LM4040-10.0, symbol LM4040
- removed D?: LM4040-5.0, symbol LM4040
- removed Q? (x4): PMP4201, MyModules:SOT363-JRL, symbol PMP4201
- removed Q? (x2): MMBF4391LT1G, symbol MMBF4391LT1G
- removed Q? (x5): MMBT3904, SOT-23, symbol MMBT3904
- removed Q? (x2): MMBT3906, SOT-23, symbol MMBT3906
- removed R? (x9): 10K, MyModules:SM0603-R-JRL, symbol R_US
- removed R? (x2): 1M, MyModules:SM0603-R-JRL, symbol R_US
- removed R? (x2): 56K, MyModules:SM0603-R-JRL, symbol R_US
- removed R? (x2): 91K, MyModules:SM0603-R-JRL, symbol R_US
- removed R? (x2): 270, MyModules:SM0603-R-JRL, symbol R_US
- removed R? (x7): 4.7K, MyModules:SM0603-R-JRL, symbol R_US
- removed R? (x2): 1.8K, MyModules:SM0603-R-JRL, symbol R_US
- removed R? (x6): 10k, MyModules:SM0603-R-JRL, symbol R_US
- removed R? (x2): 2.4K, MyModules:SM0603-R-JRL, symbol R_US
- removed R? (x5): 15K, MyModules:SM0603-R-JRL, symbol R_US
- removed R? (x4): 30K, MyModules:SM0603-R-JRL, symbol R_US
- removed R? (x11): 22K, MyModules:SM0603-R-JRL, symbol R_US
- removed R? (x12): 100K, MyModules:SM0603-R-JRL, symbol R_US
- removed R?: 33K, MyModules:SM0603-R-JRL, symbol R_US
- removed R?: 39K, MyModules:SM0603-R-JRL, symbol R_US
- removed R?: 120K, MyModules:SM0603-R-JRL, symbol R_US
- removed R?: 240K, MyModules:SM0603-R-JRL, symbol R_US
- removed R?: 47K, MyModules:SM0603-R-JRL, symbol R_US
- removed R? (x4): 2.2K, MyModules:SM0603-R-JRL, symbol R_US
- removed TC? (x2): 1K 3300ppm/K, symbol R_TEMPCO
- removed U? (x12): TL072-, MyModules:TSSOP8-JRL, symbol TL072-
- removed U?: RC4558, MyModules:TSSOP8-JRL, symbol TL072-
- removed U? (x2): CD4052, symbol CD4052
- removed VR? (x2): 20K, symbol POT_US
- added D? (x2): 1N4148, symbol D
- added Q?: MMBT3906, SOT-23, symbol MMBT3906
- added Q? (x2): MMBT3904, SOT-23, symbol MMBT3904
- added Q?: J112, symbol Q_NJFET_SDG
- added R? (x2): 12K, MyModules:SM0603-R-JRL, symbol R_US
- added R? (x4): 68K, MyModules:SM0603-R-JRL, symbol R_US
- added R? (x2): 330, MyModules:SM0603-R-JRL, symbol R_US
- added R?: 470K, MyModules:SM0603-R-JRL, symbol R_US
- added R?: 82K, MyModules:SM0603-R-JRL, symbol R_US
- added R? (x4): 100K, MyModules:SM0603-R-JRL, symbol R_US
- added R?: 150K, MyModules:SM0603-R-JRL, symbol R_US
- added R?: 1meg, MyModules:SM0603-R-JRL, symbol R_US
- added R? (x2): 10K, MyModules:SM0603-R-JRL, symbol R_US
- added TP?: TEST_POINT, symbol TEST_POINT
- added U?: LM13700, symbol LM13700
- added U?: TL072-, MyModules:TSSOP8-JRL, symbol TL072-
Connections:
- net +12V: now also R?.2, R?.2
- net ENV_1: now also R?.1, R?.1, R?.2; no longer R?.1
- net ENV_2: now also R?.2
- net GND: now also D?.2 (A), Q?.1 (B), Q?.2 (E), Q?.2 (E), R?.1, R?.1
- net VCO1_XMOD: now also U?.5
- net VCO2: now also R?.1
- net ENV: now reaches R?.2, U?.3 (+)
- net ENV: now also R?.1, R?.1, R?.1, TP?.1
- new net: Q?.3 (C), U?.1
- new net: R?.1, U?.2
- new net: R?.2, R?.2, U?.3 (+)
- new net: R?.1, R?.2, U?.4 (-)
- new net: Q?.2 (E), R?.2
- new net: Q?.3 (C), R?.1, R?.2 (x2)
- new net: Q?.1 (B), R?.2
- new net: Q?.1 (S), R?.1, R?.2, U?.1
- new net: R?.1, R?.2, U?.2 (-)
- new net: R?.2, U?.3 (+)
- new net: Q?.2 (D), R?.2
- new net: D?.1 (K), R?.1
- new net: D?.2 (A), Q?.3 (G), R?.1
- new net: Q?.1 (B), R?.1
- new net CROSSMOD: R?.1
- new net XMOD_BAL: R?.2
- no-connect marks 19 -> 8
Other:
- note added: "'LEVEL' is stepped LFO \nmodulation offset and controlled\nby 'VCA LEVEL' CV - see MCB\n"
- note added: "(100K)\n"
- note added: "12 dB/oct\n"
- note added: "24 dB/oct\n"
- note added: "CROSS MODULATION"
- note added: "ENV 1 is biased up?"
- note added: "HPF"
- note added: "LFO modulation generated \nfrom one VCA on each module\ncontroller board (2 MCBs for\n2 part timbrality)"
- note added: "PULSE WIDTH MODULATION"
- note added: "SIMULATE VCF CONTROL\nneed to change to low\noffset low Iabc configuration"
- note added: "VC MIXER"
- note added: "VCA"
- note added: "VCF"
- note added: "VCF MODULATION"
- note added: "VCO MODULATION"
- note added: "VOICE MODULE"
- note removed: "No reference voltage \nhere. May need to adjust R"
- note removed: "SIMULATE VCF CONTROL"
- note removed: "ideally replace pot \nwith fixed resistor"
- note removed: "or MMBF4393?"
- note removed: "set initial pitch"
- moved on the sheet: C?, D?, Q?, R?, TP?, U?A, U?B, U?C

Commit message: working on a cross talk reduction circuit for CD4053. Seems pointless as it only works with unipolar signals. Try again another day stupid
Parts:
- removed Q?: MMBT3904, SOT-23, symbol MMBT3904
- removed R? (x2): 68K, MyModules:SM0603-R-JRL, symbol R_US
- removed R? (x3): 100K, MyModules:SM0603-R-JRL, symbol R_US
- removed R? (x3): 10K, MyModules:SM0603-R-JRL, symbol R_US
- removed U? (x2): TL072-, MyModules:TSSOP8-JRL, symbol TL072-
- added Q? (x2): 2N7002, symbol 2N7002
- added Q? (x2): MMBT3904, SOT-23, symbol MMBT3904
- added R?: 68K, MyModules:SM0603-R-JRL, symbol R_US
- added R? (x5): 10K, MyModules:SM0603-R-JRL, symbol R_US
Connections:
- net +12V: now also R?.2, R?.2
- net ENV_1: now also Q?.1 (S), R?.2
- net GND: now also Q?.2 (E), Q?.2 (E), Q?.6 (D), Q?.6 (D)
- net VCO1_MOD_SW: now also Q?.2 (G), R?.2; no longer U?.10 (S)
- net VCO2_MOD_SW: now also Q?.2 (G), R?.2; no longer U?.11 (S)
- net at Q?.5 (B2), R?.1, TP?.1: no longer R?.2
- net at R?.1: now also D?.1 (K), R?.2
- net ENV_SEL: now reaches D?.1 (K)
- net ENV_SEL: now also R?.1
- net at R?.2, U?.2 (Y0): now also Q?.1 (S)
- net at C?.2, R?.1, R?.2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: now also R?.1
- net at U?.12 (Y0): now also Q?.1 (S), R?.2
- new net: Q?.1 (B), R?.1 (x2)
- new net: Q?.3 (C), R?.1, U?.10 (S)
- new net: Q?.3 (C), R?.1, U?.11 (S)
Other:
- note added: "CD4053s are separate ICs\non JP8 module board.\nBecause of cross talk?"
- note added: "Crosstalk reduction circuit\nUntested."
- note added: "VCO PITCH MODULATION"
- note removed: "ENV 1 is biased up?"
- note removed: "VCO MODULATION"
- moved on the sheet: C?, D?, Q?, R?, TP?, U?A, U?B, U?C

Commit message: module board schematic basically captured. Need to doublecheck and confirm and try to simulation of VCA and VCF control
Parts:
- removed Q? (x2): 2N7002, symbol 2N7002
- removed Q? (x2): MMBT3904, SOT-23, symbol MMBT3904
- removed R? (x4): 10K, MyModules:SM0603-R-JRL, symbol R_US
Connections:
- net VCO1_MOD_SW: now also U?.10 (S)
- net VCO2_MOD_SW: now also U?.11 (S)
Other:
- note added: "CD4066 instead using\nextra swtiches to shunt inputs\nto minimize crosstalk?"
- note removed: "Crosstalk reduction circuit\nUntested."
- note removed: "These are separate ICs\non JP8 module board.\nBecause of cross talk?"
- moved on the sheet: C?, Q?, R?, U?A, U?B, U?C

Commit message: updating VCF control with notes from simulation
Parts:
- R?: value 68K -> 27K
- R?: value 100K -> 22K
Connections:
- net at R?.2, U?.3 (+): now also R?.2
- net at R?.2, U?.4 (-): no longer R?.2
- net at R?.2: now also Q?.5 (B2), R?.1, TP?.1
Other:
- note added: "ENV_SEL needs to swing from \n+ve to -ve rail, so use comparator \nhere?"
- note added: "J112 Vgs(on) isn't low enough to block\n-ve inverted envelope voltages with -12V\ngate. Lower ENV amplitude or find different FET?\n"
- note added: "Simulated. Need to investigate \nfurther and test original JP8\nVCA modulation behaviour.\nNot getting good offness \nwhen LEVEL CV is 0V."
- moved on the sheet: R?, U?A
Changed lines of the file:
@@
 L R_US R?
 U 1 1 57F765F7
-P 9075 16825
-F 0 "R?" H 8975 16800 50  0000 C CNN
-F 1 "100K" H 8950 16875 50  0000 C CNN
-F 2 "MyModules:SM0603-R-JRL" H 9075 16825 60  0001 C CNN
-F 3 "" H 9075 16825 60  0001 C CNN
-F 4 "P10.0KCCT-ND" V 9075 16825 60  0001 C CNN "Digikey"
-	1    9075 16825
+P 9075 17125
+F 0 "R?" H 8975 17100 50  0000 C CNN
+F 1 "100K" H 8950 17175 50  0000 C CNN
+F 2 "MyModules:SM0603-R-JRL" H 9075 17125 60  0001 C CNN
+F 3 "" H 9075 17125 60  0001 C CNN
+F 4 "P10.0KCCT-ND" V 9075 17125 60  0001 C CNN "Digikey"
+	1    9075 17125
 	1    0    0    1
 $EndComp
@@
 P 14875 16625
 F 0 "R?" V 14950 16775 50  0000 C CNN
-F 1 "68K" V 14950 16450 50  0000 C CNN
+F 1 "27K" V 14950 16450 50  0000 C CNN
 F 2 "MyModules:SM0603-R-JRL" H 14875 16625 60  0001 C CNN
 F 3 "" H 14875 16625 60  0001 C CNN
@@
 L R_US R?
 U 1 1 57FABB71
-P 10800 16375
-F 0 "R?" V 10875 16525 50  0000 C CNN
-F 1 "68K" V 10875 16200 50  0000 C CNN
-F 2 "MyModules:SM0603-R-JRL" H 10800 16375 60  0001 C CNN
-F 3 "" H 10800 16375 60  0001 C CNN
-F 4 "P10.0KCCT-ND" V 10800 16375 60  0001 C CNN "Digikey"
-	1    10800 16375
+P 10650 16675
+F 0 "R?" V 10725 16825 50  0000 C CNN
+F 1 "68K" V 10725 16500 50  0000 C CNN
+F 2 "MyModules:SM0603-R-JRL" H 10650 16675 60  0001 C CNN
+F 3 "" H 10650 16675 60  0001 C CNN
+F 4 "P10.0KCCT-ND" V 10650 16675 60  0001 C CNN "Digikey"
+	1    10650 16675
 	0    -1   -1   0
 $EndComp
@@
 L TL072- U?
 U 1 1 57FC4FC2
-P 9650 16375
-F 0 "U?" H 9600 16575 60  0000 L CNN
-F 1 "TL072-" H 9775 16250 60  0000 L CNN
-F 2 "MyModules:TSSOP8-JRL" H 9650 16375 60  0001 C CNN
-F 3 "~" H 9650 16375 60  0000 C CNN
-	1    9650 16375
-	1    0    0    -1
-$EndComp
-Text GLabel 8475 16475 0    60   Input ~ 0
+P 9650 16675
+F 0 "U?" H 9600 16875 60  0000 L CNN
+F 1 "TL072-" H 9775 16550 60  0000 L CNN
+F 2 "MyModules:TSSOP8-JRL" H 9650 16675 60  0001 C CNN
+F 3 "~" H 9650 16675 60  0000 C CNN
+	1    9650 16675
+	1    0    0    -1
+$EndComp
+Text GLabel 8475 16775 0    60   Input ~ 0
 KCV_1
 $Comp
 L R_US R?
 U 1 1 57FCF9D4
-P 8800 16475
-F 0 "R?" V 8875 16625 50  0000 C CNN
-F 1 "100K" V 8875 16300 50  0000 C CNN
-F 2 "MyModules:SM0603-R-JRL" H 8800 16475 60  0001 C CNN
-F 3 "" H 8800 16475 60  0001 C CNN
-F 4 "P10.0KCCT-ND" V 8800 16475 60  0001 C CNN "Digikey"
-	1    8800 16475
+P 8800 16775
+F 0 "R?" V 8875 16925 50  0000 C CNN
+F 1 "100K" V 8875 16600 50  0000 C CNN
+F 2 "MyModules:SM0603-R-JRL" H 8800 16775 60  0001 C CNN
+F 3 "" H 8800 16775 60  0001 C CNN
+F 4 "P10.0KCCT-ND" V 8800 16775 60  0001 C CNN "Digikey"
+	1    8800 16775
 	0    -1   1    0
 $EndComp
-Text GLabel 8475 16275 0    60   Input ~ 0
+Text GLabel 8475 16575 0    60   Input ~ 0
 VCO1_RANGE
 $Comp
 L R_US R?
 U 1 1 57FD14AF
-P 8800 16275
-F 0 "R?" V 8875 16425 50  0000 C CNN
-F 1 "100K" V 8875 16100 50  0000 C CNN
-F 2 "MyModules:SM0603-R-JRL" H 8800 16275 60  0001 C CNN
-F 3 "" H 8800 16275 60  0001 C CNN
-F 4 "P10.0KCCT-ND" V 8800 16275 60  0001 C CNN "Digikey"
-	1    8800 16275
+P 8800 16575
+F 0 "R?" V 8875 16725 50  0000 C CNN
+F 1 "100K" V 8875 16400 50  0000 C CNN
+F 2 "MyModules:SM0603-R-JRL" H 8800 16575 60  0001 C CNN
+F 3 "" H 8800 16575 60  0001 C CNN
+F 4 "P10.0KCCT-ND" V 8800 16575 60  0001 C CNN "Digikey"
+	1    8800 16575
 	0    -1   -1   0
 $EndComp
@@
 L GND_R #PWR?
 U 1 1 57FD1DA6
-P 9075 17075
-F 0 "#PWR?" H 9075 17075 30  0001 C CNN
-F 1 "GND_R" H 9075 16975 30  0001 C CNN
-F 2 "" H 9075 17075 60  0000 C CNN
-F 3 "" H 9075 17075 60  0000 C CNN
-	1    9075 17075
+P 9075 17375
+F 0 "#PWR?" H 9075 17375 30  0001 C CNN
+F 1 "GND_R" H 9075 17275 30  0001 C CNN
+F 2 "" H 9075 17375 60  0000 C CNN
+F 3 "" H 9075 17375 60  0000 C CNN
+	1    9075 17375
 	1    0    0    -1
 $EndComp
@@
 L R_US R?
 U 1 1 57FD5870
-P 9600 15725
-F 0 "R?" V 9675 15875 50  0000 C CNN
-F 1 "100K" V 9675 15550 50  0000 C CNN
-F 2 "MyModules:SM0603-R-JRL" H 9600 15725 60  0001 C CNN
-F 3 "" H 9600 15725 60  0001 C CNN
-F 4 "P10.0KCCT-ND" V 9600 15725 60  0001 C CNN "Digikey"
-	1    9600 15725
+P 9600 16025
+F 0 "R?" V 9675 16175 50  0000 C CNN
+F 1 "100K" V 9675 15850 50  0000 C CNN
+F 2 "MyModules:SM0603-R-JRL" H 9600 16025 60  0001 C CNN
+F 3 "" H 9600 16025 60  0001 C CNN
+F 4 "P10.0KCCT-ND" V 9600 16025 60  0001 C CNN "Digikey"
+	1    9600 16025
 	0    -1   -1   0
 $EndComp
@@
 Wire Wire Line
 	15475 3575 15475 4500
-Connection ~ 9075 16275
-Wire Wire Line
-	9075 15725 9075 16275
-Wire Wire Line
-	9400 15725 9075 15725
-Connection ~ 10200 16375
-Wire Wire Line
-	10200 15725 10200 16375
-Wire Wire Line
-	9800 15725 10200 15725
-Wire Wire Line
-	9075 17025 9075 17075
-Connection ~ 9075 16475
-Wire Wire Line
-	9075 16625 9075 16475
-Wire Wire Line
-	8600 16275 8475 16275
-Wire Wire Line
-	9000 16275 9150 16275
-Wire Wire Line
-	8600 16475 8475 16475
-Wire Wire Line
-	9000 16475 9150 16475
-Wire Wire Line
-	10150 16375 10600 16375
+Connection ~ 9075 16575
+Wire Wire Line
+	9075 16025 9075 16575
+Wire Wire Line
+	9400 16025 9075 16025
+Connection ~ 10200 16675
+Wire Wire Line
+	10200 16025 10200 16675
+Wire Wire Line
+	9800 16025 10200 16025
+Wire Wire Line
+	9075 17325 9075 17375
+Connection ~ 9075 16775
+Wire Wire Line
+	9075 16925 9075 16775
+Wire Wire Line
+	8600 16575 8475 16575
+Wire Wire Line
+	9000 16575 9150 16575
+Wire Wire Line
+	8600 16775 8475 16775
+Wire Wire Line
+	9000 16775 9150 16775
+Wire Wire Line
+	10150 16675 10450 16675
 Wire Wire Line
 	17400 16000 18300 16000
-Connection ~ 11100 16375
 Wire Wire Line
 	12525 19025 11950 19025
@@
 	11675 15725 11675 15800
 Wire Wire Line
-	11450 16675 11850 16675
+	10850 16675 11850 16675
 Wire Wire Line
 	11450 16750 11450 16675
-Wire Wire Line
-	11000 16375 11850 16375
 Wire Wire Line
 	11100 16375 11100 16750
@@
 	17400 16000 17400 16375
 Wire Wire Line
-	15100 16625 17050 16625
+	15075 16625 17050 16625
 Wire Wire Line
 	18350 18125 18350 16275
@@
 	14500 7900 14350 7900
 Wire Wire Line
-	14350 7900 14350 8450
-Wire Wire Line
-	14350 8450 13425 8450
+	14350 8450 14350 7900
+Wire Wire Line
+	13425 8450 14350 8450
 $Comp
 L R_US R?
@@
 P 15450 20775
 F 0 "R?" V 15525 20925 50  0000 C CNN
-F 1 "100K" V 15525 20600 50  0000 C CNN
+F 1 "22K" V 15525 20600 50  0000 C CNN
 F 2 "MyModules:SM0603-R-JRL" H 15450 20775 60  0001 C CNN
 F 3 "" H 15450 20775 60  0001 C CNN
@@
 Wire Wire Line
 	19800 4050 19950 4050
+Text Notes 29200 16850 0    60   ~ 0
+Simulated. Need to investigate \nfurther and test original JP8\nVCA modulation behaviour.\nNot getting good offness \nwhen LEVEL CV is 0V.
+Connection ~ 11450 16675
+Wire Wire Line
+	11850 16375 11100 16375
+Text Notes 16225 20050 0    60   ~ 0
+J112 Vgs(on) isn't low enough to block\n-ve inverted envelope voltages with -12V\ngate. Lower ENV amplitude or find different FET?\n
+Text Notes 13350 21125 0    60   ~ 0
+ENV_SEL needs to swing from \n+ve to -ve rail, so use comparator \nhere?
 $EndSCHEMATC
