File: voice.sch (KiCad schematic (older format))
At the start: 187 parts

Commit message: changed notes to reflect observations from SPICE simulation of VCF envelope switching
Other:
- note added: "ENV_SEL needs to swing close\n+ve and -ve rail. To keep JFET off\nneed <= -11V."
- note added: "J112 Vgs(off) isn't low enough to block\n-ve inverted envelope voltages with -11V\ngate. Lower ENV amplitude or find different FET?\nON Semi TF412S has low Vgs{off) - will probably work\n2SK932 also looks promising\n"
- note added: "Maybe JFET shunts here?"
- note added: "Probably need to use a lower Vgs(off) FET\nthan J112 here as in VCF envelope modulation\nselector circuit."
- note removed: "CD4066 instead using\nextra swtiches to shunt inputs\nto minimize crosstalk?"
- note removed: "ENV_SEL needs to swing from \n+ve to -ve rail, so use comparator \nhere?"
- note removed: "J112 Vgs(on) isn't low enough to block\n-ve inverted envelope voltages with -12V\ngate. Lower ENV amplitude or find different FET?\n"
Changed lines of the file:
@@
 	14500 7900 14350 7900
 Wire Wire Line
-	14350 8450 14350 7900
-Wire Wire Line
-	13425 8450 14350 8450
+	14350 7900 14350 8450
+Wire Wire Line
+	14350 8450 13425 8450
 $Comp
 L R_US R?
@@
 Wire Wire Line
 	18625 3850 19250 3850
-Connection ~ 18850 3850
 Text Notes 19475 3150 0    60   ~ 0
 CD4053s are separate ICs\non JP8 module board.\nBecause of cross talk?
-Text Notes 17775 4300 0    60   ~ 0
-CD4066 instead using\nextra swtiches to shunt inputs\nto minimize crosstalk?
+Text Notes 17950 4075 0    60   ~ 0
+Maybe JFET shunts here?
 Wire Wire Line
 	19075 2500 19225 2500
@@
 Wire Wire Line
 	11850 16375 11100 16375
-Text Notes 16225 20050 0    60   ~ 0
-J112 Vgs(on) isn't low enough to block\n-ve inverted envelope voltages with -12V\ngate. Lower ENV amplitude or find different FET?\n
+Text Notes 16225 20175 0    60   ~ 0
+J112 Vgs(off) isn't low enough to block\n-ve inverted envelope voltages with -11V\ngate. Lower ENV amplitude or find different FET?\nON Semi TF412S has low Vgs{off) - will probably work\n2SK932 also looks promising\n
 Text Notes 13350 21125 0    60   ~ 0
-ENV_SEL needs to swing from \n+ve to -ve rail, so use comparator \nhere?
+ENV_SEL needs to swing close\n+ve and -ve rail. To keep JFET off\nneed <= -11V.
+Text Notes 24800 17225 0    60   ~ 0
+Probably need to use a lower Vgs(off) FET\nthan J112 here as in VCF envelope modulation\nselector circuit.
 $EndSCHEMATC

Commit message: made some notes about VCA control after studying actual JP8. Updated proposd panel layout
Parts:
- U? (x2): value TL072- -> RC4558
Other:
- note added: "OFFSET"
- note added: "When LEVEL CV = 0V there is some\nbleedthrough of ENV_2 signal. When LEVEL CV < 0V\nthen there is no output. Amount of bleedthrough varies \nfrom voice to voice of JP8\n"
Changed lines of the file:
@@
 P 13975 16625
 F 0 "U?" H 13925 16825 60  0000 L CNN
-F 1 "TL072-" H 14100 16500 60  0000 L CNN
+F 1 "RC4558" H 14100 16500 60  0000 L CNN
 F 2 "MyModules:TSSOP8-JRL" H 13975 16625 60  0001 C CNN
 F 3 "~" H 13975 16625 60  0000 C CNN
@@
 P 9650 16675
 F 0 "U?" H 9600 16875 60  0000 L CNN
-F 1 "TL072-" H 9775 16550 60  0000 L CNN
+F 1 "RC4558" H 9775 16550 60  0000 L CNN
 F 2 "MyModules:TSSOP8-JRL" H 9650 16675 60  0001 C CNN
 F 3 "~" H 9650 16675 60  0000 C CNN
@@
 Text Notes 24800 17225 0    60   ~ 0
 Probably need to use a lower Vgs(off) FET\nthan J112 here as in VCF envelope modulation\nselector circuit.
+Text Notes 29200 17325 0    60   ~ 0
+When LEVEL CV = 0V there is some\nbleedthrough of ENV_2 signal. When LEVEL CV < 0V\nthen there is no output. Amount of bleedthrough varies \nfrom voice to voice of JP8\n
+Text Notes 14275 15325 2    60   ~ 0
+OFFSET
+Text Notes 28850 13925 2    60   ~ 0
+OFFSET
+Text Notes 17300 1875 2    60   ~ 0
+OFFSET
+Text Notes 23500 2525 2    60   ~ 0
+OFFSET
 $EndSCHEMATC

Commit message: gathering switch, CV and modulation inputs from voice
Parts:
- added Q?: MMBT3906, SOT-23, symbol MMBT3906
- added R?: 22K, MyModules:SM0603-R-JRL, symbol R_US
Connections:
- net GND: now also Q?.1 (B)
- net PWM: no longer R?.1
- net RES_CTRL: now also R?.1; no longer U?.1
- new net: Q?.3 (C), U?.1
- new net: Q?.2 (E), R?.2
- new net PWM_LEVEL: R?.1
Other:
- note added: "-11V to +12V"
- note added: "-11V to +12V switch"
- note added: "10V switch"
- note added: "15K - 25K\n"
- note added: "5V"
- note added: "COMMON\n"
- note added: "CV"
- note added: "MODULATION"
- note added: "OUTPUT"
- note added: "VOICE"
Changed lines of the file:
@@
 $EndComp
 Text GLabel 16675 8525 0    60   Input ~ 0
-PWM
+PWM_LEVEL
 $Comp
 L R_US R?
@@
 	-1   0    0    1
 $EndComp
-Text GLabel 27500 11775 2    60   Input ~ 0
+Text GLabel 28725 11775 2    60   Input ~ 0
 RES_CTRL
 $Comp
@@
 56K - 100K
 $Sheet
-S 6000 1575 2050 1700
+S 4975 1600 2250 1875
 U 57F5D1D5
 F0 "Envelopes" 60
@@
 	26250 12175 26250 10675
 Wire Wire Line
-	27250 11775 27500 11775
+	27250 11775 27825 11775
 Wire Wire Line
 	27250 12275 27250 11775
@@
 Text Notes 23500 2525 2    60   ~ 0
 OFFSET
+Text Notes 13725 20700 0    60   ~ 0
+-11V to +12V
+Text Notes 25975 16775 0    60   ~ 0
+-11V to +12V
+Text Notes 14850 2600 2    60   ~ 0
+OFFSET
+Text Notes 7500 5625 2    60   ~ 0
+OFFSET
+Text GLabel 7725 5750 0    60   Input ~ 0
+VCO_ENV_MOD_BAL
+Text GLabel 7725 5900 0    60   Input ~ 0
+VCO_MOD_BAL
+Text Notes 3875 5625 2    60   ~ 0
+-11V to +12V switch
+Text Notes 2475 5600 2    60   ~ 0
+10V switch
+Text Notes 4800 5625 2    60   ~ 0
+MODULATION
+Text Notes 5375 5625 2    60   ~ 0
+CV
+Text Notes 8500 5625 2    60   ~ 0
+OUTPUT
+Text GLabel 5650 5750 0    60   Input ~ 0
+VCO_ENV_MOD
+Text GLabel 4775 5750 0    60   Input ~ 0
+VCO_LFO_MOD
+Text GLabel 2600 5750 0    60   Input ~ 0
+VCO1_MOD_SW
+Text GLabel 2600 5900 0    60   Input ~ 0
+VCO2_MOD_SW
+Text GLabel 7725 6050 0    60   Input ~ 0
+XMOD_BAL
+Text GLabel 5625 5900 0    60   Input ~ 0
+CROSSMOD
+Text GLabel 4775 5900 0    60   Input ~ 0
+LFO
+Text GLabel 2600 6050 0    60   Input ~ 0
+PWM_SEL
+Text GLabel 2600 6200 0    60   Input ~ 0
+PW/PWM
+Text GLabel 5625 6050 0    60   Input ~ 0
+PWM_LEVEL
+Text GLabel 5625 6200 0    60   Input ~ 0
+VCO1_LEVEL
+Text GLabel 5625 6350 0    60   Input ~ 0
+VCO2_LEVEL
+$Comp
+L MMBT3906 Q?
+U 1 1 5809D2EC
+P 28025 11875
+F 0 "Q?" H 28225 11950 50  0000 L CNN
+F 1 "MMBT3906" H 27650 12100 50  0000 L CNN
+F 2 "SOT-23" H 28225 11800 50  0001 L CIN
+F 3 "" H 28025 11875 50  0000 L CNN
+	1    28025 11875
+	0    -1   -1   0
+$EndComp
+$Comp
+L GND_R #PWR?
+U 1 1 5809EC98
+P 28025 12075
+F 0 "#PWR?" H 28025 12075 30  0001 C CNN
+F 1 "GND_R" H 28025 11975 30  0001 C CNN
+F 2 "" H 28025 12075 60  0000 C CNN
+F 3 "" H 28025 12075 60  0000 C CNN
+	1    28025 12075
+	1    0    0    -1
+$EndComp
+$Comp
+L R_US R?
+U 1 1 5809F49E
+P 28475 11775
+F 0 "R?" V 28555 11775 50  0000 C CNN
+F 1 "22K" V 28395 11775 50  0000 C CNN
+F 2 "MyModules:SM0603-R-JRL" H 28475 11775 60  0001 C CNN
+F 3 "~" H 28475 11775 60  0000 C CNN
+	1    28475 11775
+	0    1    -1   0
+$EndComp
+Wire Wire Line
+	28275 11775 28225 11775
+Wire Wire Line
+	28675 11775 28725 11775
+Text Notes 28275 11975 0    50   ~ 0
+15K - 25K\n
+Text GLabel 5625 6500 0    60   Input ~ 0
+RES_CTRL
+Text GLabel 8200 5750 2    60   Output ~ 0
+OUT
+Text GLabel 7725 6200 0    60   Input ~ 0
+VCA_BAL
+Text GLabel 3600 5750 0    60   Input ~ 0
+VCF_12dB
+Text GLabel 3600 5900 0    60   Input ~ 0
+VCF_24dB
+Text GLabel 4775 6050 0    60   Input ~ 0
+LEVEL
+Text GLabel 3600 6050 0    60   Input ~ 0
+ENV_SEL
+Text GLabel 7725 6350 0    60   Input ~ 0
+VCF_TUNE
+Text GLabel 5625 6650 0    60   Input ~ 0
+VCF_KF
+Text GLabel 4775 6200 0    60   Input ~ 0
+VCF_CUTOFF
+Text GLabel 5625 6800 0    60   Input ~ 0
+VCF_ENV_MOD
+Text GLabel 1275 5750 0    60   Input ~ 0
+VCO1_RANGE
+Text GLabel 6650 6050 0    60   Input ~ 0
+VCO1_TUNE
+Text GLabel 8200 5900 2    60   Output ~ 0
+VCO1_AUTOTUNE
+Text GLabel 8200 6050 2    60   Output ~ 0
+VCO2_AUTOTUNE
+Text GLabel 1675 5750 0    60   Input ~ 0
+GATE
+Text Notes 1600 5600 2    60   ~ 0
+5V
+Text GLabel 2600 6350 0    60   Input ~ 0
+VCO1_WF-0
+Text GLabel 2600 6500 0    60   Input ~ 0
+VCO1_WF-1
+Text GLabel 2600 6650 0    60   Input ~ 0
+VCO2_WF-0
+Text GLabel 2600 6800 0    60   Input ~ 0
+VCO2_WF-1
+Text GLabel 1275 5925 0    60   Input ~ 0
+NOISE
+Text GLabel 5625 7250 0    60   Input ~ 0
+ENV1_R
+Text GLabel 5625 7400 0    60   Input ~ 0
+ENV1_S
+Text GLabel 5625 7100 0    60   Input ~ 0
+ENV1_D
+Text GLabel 5625 6950 0    60   Input ~ 0
+ENV1_A
+Text GLabel 5625 7850 0    60   Input ~ 0
+ENV2_R
+Text GLabel 5625 8000 0    60   Input ~ 0
+ENV2_S
+Text GLabel 5625 7700 0    60   Input ~ 0
+ENV2_D
+Text GLabel 5625 7550 0    60   Input ~ 0
+ENV2_A
+Text GLabel 2600 6950 0    60   Input ~ 0
+SYNC_CTRL
+Text Notes 6925 5450 2    60   ~ 0
+VOICE
+Text GLabel 6650 5750 0    60   Input ~ 0
+KCV_1
+Text GLabel 6650 5900 0    60   Input ~ 0
+KCV_2
+Text GLabel 6650 6200 0    60   Input ~ 0
+VCO2_TUNE
+Text Notes 5075 5450 2    60   ~ 0
+COMMON\n
+Text Notes 6450 5625 2    60   ~ 0
+CV
 $EndSCHEMATC

Commit message: found Toshiba single op amp equivalent of RC4558. Starting to pair off and power op amps and OTAs
Parts:
- removed U? (x2): TL072-, MyModules:TSSOP8-JRL, symbol TL072-
- removed U? (x2): RC4558, MyModules:TSSOP8-JRL, symbol TL072-
- added U? (x3): TA75S558F, symbol TA75S558F
- added U?: TS321, symbol TS321
Connections:
- net +12V: now also U?.11 (V+), U?.11 (V+), U?.11 (V+), U?.11 (V+), U?.8 (V+), U?.5 (V+), U?.5 (V+), U?.5 (V+), U?.5 (V+); no longer U?.6 (V-)
- net -12V: now also U?.4 (V-), U?.6 (V-), U?.6 (V-), U?.6 (V-), U?.6 (V-), U?.2 (V-), U?.2 (V-), U?.2 (V-), U?.2 (V-); no longer U?.11 (V+)
- net GND: now also U?.5 (+), U?.1 (+), U?.1 (+), U?.1 (+), U?.3 (+); no longer U?.3 (+)
- net PWM: now also U?.4
- net at C?.1, R?.1, R?.2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: now also U?.3 (-)
- net at C?.1, R?.1, U?.5: now also U?.3 (-)
- net at C?.2, R?.1, R?.2: now also U?.4
- net at Q?.3 (C): now also U?.16; no longer U?.1 (x3)
- net at R?.1: now also U?.15; no longer U?.2 (x2)
- net at R?.2, R?.2: now also U?.14 (+); no longer U?.3 (+) (x2)
- net at R?.2: now also U?.13 (-); no longer U?.4 (-) (x2)
- net at Q?.2 (E): now also U?.12; no longer U?.5
- net at R?.1, R?.1, R?.1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: now also U?.12, U?.6 (-); no longer U?.2 (-), U?.5
- net at R?.1, R?.2: now also U?.7; no longer U?.1
- net at R?.2, R?.2, R?.2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: now also U?.12; no longer U?.5
- net at R?.1, R?.2: now also U?.13 (-); no longer U?.4 (-)
- net at R?.1, R?.1: now also U?.14 (+); no longer U?.3 (+)
- net at C?.2, Q?.6 (C1), R?.1: now also U?.4 (-)
- net at C?.1, R?.2: now also U?.1
- net at C?.2, R?.1, R?.1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: now also U?.4
- net at C?.1, R?.1, R?.1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: now also U?.3 (-)
Other:
- note added: "(BIPOLAR)"
- note added: "Toshiba TA75S558F seems like\nSC74A/SOT573 single equivalent\nto RC4558"

Commit message: had annotation of ICs started
Parts:
- added unit 2 of U14
- added unit 2 of U17
- gave numbers to parts that had none: 15
Connections:
- net +12V: now also U10.11 (V+), U14.11 (V+)
- net -12V: now also U10.6 (V-), U14.6 (V-)
- net GND: now also U17.5 (+)
- net VCO1_XMOD: now also U10.12; no longer U10.5
- net at Q?.3 (C): now also U10.16; no longer U10.1
- net at R?.1: now also U10.15; no longer U10.2
- net at R?.2, R?.2: now also U10.14 (+); no longer U10.3 (+)
- net at R?.1, R?.2: now also U10.13 (-); no longer U10.4 (-)
- new net: U17.6 (-), U17.7
- no-connect marks 8 -> 18
Other:
- moved on the sheet: C?, D?, Q?, R?, TP?, U15A, U15B, U16A, U17A, U18A, U18B, U19A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

Commit message: sorting out packages, also taking deeper look at saw to tri converter. there are problems on 12V power and 10V saw that need to be sorted. NPN in tri converter is a an ultra fast switcher that might be hard to find an equiavalent for. Worth looking at tri waveform out of converter on JP8
Parts:
- removed Q? (x8): J112, symbol Q_NJFET_SDG
- added Q? (x5): J112, MyModules:SOT23-132-JRL, symbol Q_NJFET_DSG
- added Q? (x3): J201, MyModules:SOT23-132-JRL, symbol Q_NJFET_DSG
Connections:
- net +12V: now also Q?.1 (D), Q?.1 (D), Q?.1 (D), Q?.1 (D), Q?.1 (D)
- net ENV_1: now also Q?.2 (S)
- net at C?.1, U16.5: now also Q?.3 (G)
- net at C?.2, R?.1, R?.2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: now also Q?.2 (S)
- net at R?.2: now also Q?.1 (D)
- net at D?.2 (A), R?.1: now also Q?.3 (G) (x3)
- net at C?.1, U18.5: now also Q?.3 (G)
- net at R?.1, R?.2, R?.2: now also Q?.2 (S) (x2)
- net at C?.1, U18.12: now also Q?.3 (G)
- net at R?.1, R?.2, R?.2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: now also Q?.2 (S), Q?.2 (S)
- net at C?.1, U19.12: now also Q?.3 (G)
- net at C?.1, U19.5: now also Q?.3 (G)
- net at C?.2 (-), R?.1, R?.2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: now also Q?.2 (S), Q?.2 (S)
- net at C?.2 (-): now also Q?.1 (D) (x2)
Other:
- note added: "J112 Vgs(off) isn't low enough to block\n-ve inverted envelope voltages with -11V\ngate. Lower ENV amplitude or find different FET?\nON Semi TF412S has low Vgs{off) - will probably work\n2SK932 and J201 also look promising\n"
- note removed: "J112 Vgs(off) isn't low enough to block\n-ve inverted envelope voltages with -11V\ngate. Lower ENV amplitude or find different FET?\nON Semi TF412S has low Vgs{off) - will probably work\n2SK932 also looks promising\n"
Changed lines of the file:
@@
 $EndComp
 $Comp
-L Q_NJFET_SDG Q?
-U 1 1 57F85048
-P 9900 12250
-F 0 "Q?" H 10200 12300 50  0000 R CNN
-F 1 "J112" H 10275 12225 50  0000 R CNN
-F 2 "" H 10100 12350 29  0000 C CNN
-F 3 "" H 9900 12250 60  0000 C CNN
-	1    9900 12250
-	1    0    0    -1
-$EndComp
-$Comp
 L +12V #PWR?
 U 1 1 57F8A12B
@@
 $EndComp
 $Comp
-L Q_NJFET_SDG Q?
-U 1 1 57FB3263
-P 14700 12325
-F 0 "Q?" H 15000 12375 50  0000 R CNN
-F 1 "J112" H 15075 12300 50  0000 R CNN
-F 2 "" H 14900 12425 29  0000 C CNN
-F 3 "" H 14700 12325 60  0000 C CNN
-	1    14700 12325
-	1    0    0    -1
-$EndComp
-$Comp
 L R_US R?
 U 1 1 57FBF4DE
@@
 $EndComp
 $Comp
-L Q_NJFET_SDG Q?
-U 1 1 57FBF4F5
-P 18000 12325
-F 0 "Q?" H 18300 12375 50  0000 R CNN
-F 1 "J112" H 18375 12300 50  0000 R CNN
-F 2 "" H 18200 12425 29  0000 C CNN
-F 3 "" H 18000 12325 60  0000 C CNN
-	1    18000 12325
-	1    0    0    -1
-$EndComp
-$Comp
 L R_US R?
 U 1 1 57FC414F
@@
 $EndComp
 $Comp
-L Q_NJFET_SDG Q?
-U 1 1 57FC4166
-P 21300 12325
-F 0 "Q?" H 21600 12375 50  0000 R CNN
-F 1 "J112" H 21675 12300 50  0000 R CNN
-F 2 "" H 21500 12425 29  0000 C CNN
-F 3 "" H 21300 12325 60  0000 C CNN
-	1    21300 12325
-	1    0    0    -1
-$EndComp
-$Comp
 L R_US R?
 U 1 1 57FC52F8
@@
 $EndComp
 $Comp
-L Q_NJFET_SDG Q?
-U 1 1 57FC5310
-P 24600 12325
-F 0 "Q?" H 24900 12375 50  0000 R CNN
-F 1 "J112" H 24975 12300 50  0000 R CNN
-F 2 "" H 24800 12425 29  0000 C CNN
-F 3 "" H 24600 12325 60  0000 C CNN
-	1    24600 12325
-	1    0    0    -1
-$EndComp
-$Comp
 L GND_R #PWR?
 U 1 1 57FC86EB
@@
 $EndComp
 $Comp
-L Q_NJFET_SDG Q?
-U 1 1 57FFD412
-P 25250 14800
-F 0 "Q?" H 25550 14850 50  0000 R CNN
-F 1 "J112" H 25625 14775 50  0000 R CNN
-F 2 "" H 25450 14900 29  0000 C CNN
-F 3 "" H 25250 14800 60  0000 C CNN
-	1    25250 14800
-	0    -1   -1   0
-$EndComp
-$Comp
 L R_US R?
 U 1 1 57FFEB66
@@
 $EndComp
 $Comp
-L Q_NJFET_SDG Q?
-U 1 1 58006A40
-P 25975 15800
-F 0 "Q?" H 26275 15850 50  0000 R CNN
-F 1 "J112" H 26350 15775 50  0000 R CNN
-F 2 "" H 26175 15900 29  0000 C CNN
-F 3 "" H 25975 15800 60  0000 C CNN
-	1    25975 15800
-	0    -1   -1   0
-$EndComp
-$Comp
 L R_US R?
 U 1 1 58006A46
@@
 Text Notes 13475 2275 0    150  ~ 30
 VCO PITCH MODULATION
-Text Notes 6650 16025 0    150  ~ 30
+Text Notes 6500 16175 0    150  ~ 30
 VCF MODULATION
 Text Notes 13375 6350 0    150  ~ 30
@@
 	0    -1   -1   0
 $EndComp
-$Comp
-L Q_NJFET_SDG Q?
-U 1 1 57FADB46
-P 13750 20025
-F 0 "Q?" H 14050 20075 50  0000 R CNN
-F 1 "J112" H 14125 20000 50  0000 R CNN
-F 2 "" H 13950 20125 29  0000 C CNN
-F 3 "" H 13750 20025 60  0000 C CNN
-	1    13750 20025
-	0    -1   -1   0
-$EndComp
 Wire Wire Line
 	13950 19925 14275 19925
@@
 	9450 17125 8700 17125
 Text Notes 13825 20925 0    60   ~ 0
-J112 Vgs(off) isn't low enough to block\n-ve inverted envelope voltages with -11V\ngate. Lower ENV amplitude or find different FET?\nON Semi TF412S has low Vgs{off) - will probably work\n2SK932 also looks promising\n
+J112 Vgs(off) isn't low enough to block\n-ve inverted envelope voltages with -11V\ngate. Lower ENV amplitude or find different FET?\nON Semi TF412S has low Vgs{off) - will probably work\n2SK932 and J201 also look promising\n
 Text Notes 10950 21875 0    60   ~ 0
 ENV_SEL needs to swing close\n+ve and -ve rail. To keep JFET off\nneed <= -11V.
@@
 Wire Wire Line
 	5900 14325 5900 14425
+$Comp
+L Q_NJFET_DSG Q?
+U 1 1 58111A83
+P 14700 12325
+F 0 "Q?" H 15000 12375 50  0000 R CNN
+F 1 "J112" H 15075 12300 50  0000 R CNN
+F 2 "MyModules:SOT23-132-JRL" H 14900 12425 29  0001 C CNN
+F 3 "" H 14700 12325 60  0000 C CNN
+	1    14700 12325
+	1    0    0    -1
+$EndComp
+$Comp
+L Q_NJFET_DSG Q?
+U 1 1 58112FD8
+P 9900 12250
+F 0 "Q?" H 10200 12300 50  0000 R CNN
+F 1 "J112" H 10275 12225 50  0000 R CNN
+F 2 "MyModules:SOT23-132-JRL" H 10100 12350 29  0001 C CNN
+F 3 "" H 9900 12250 60  0000 C CNN
+	1    9900 12250
+	1    0    0    -1
+$EndComp
+$Comp
+L Q_NJFET_DSG Q?
+U 1 1 58113ED6
+P 18000 12325
+F 0 "Q?" H 18300 12375 50  0000 R CNN
+F 1 "J112" H 18375 12300 50  0000 R CNN
+F 2 "MyModules:SOT23-132-JRL" H 18200 12425 29  0001 C CNN
+F 3 "" H 18000 12325 60  0000 C CNN
+	1    18000 12325
+	1    0    0    -1
+$EndComp
+$Comp
+L Q_NJFET_DSG Q?
+U 1 1 58116222
+P 21300 12325
+F 0 "Q?" H 21600 12375 50  0000 R CNN
+F 1 "J112" H 21675 12300 50  0000 R CNN
+F 2 "MyModules:SOT23-132-JRL" H 21500 12425 29  0001 C CNN
+F 3 "" H 21300 12325 60  0000 C CNN
+	1    21300 12325
+	1    0    0    -1
+$EndComp
+$Comp
+L Q_NJFET_DSG Q?
+U 1 1 58116E9A
+P 24600 12325
+F 0 "Q?" H 24900 12375 50  0000 R CNN
+F 1 "J112" H 24975 12300 50  0000 R CNN
+F 2 "MyModules:SOT23-132-JRL" H 24800 12425 29  0001 C CNN
+F 3 "" H 24600 12325 60  0000 C CNN
+	1    24600 12325
+	1    0    0    -1
+$EndComp
+$Comp
+L Q_NJFET_DSG Q?
+U 1 1 581190CB
+P 25250 14800
+F 0 "Q?" V 25575 14675 50  0000 R CNN
+F 1 "J201" V 25475 14700 50  0000 R CNN
+F 2 "MyModules:SOT23-132-JRL" H 25450 14900 29  0001 C CNN
+F 3 "" H 25250 14800 60  0000 C CNN
+	1    25250 14800
+	0    1    -1   0
+$EndComp
+$Comp
+L Q_NJFET_DSG Q?
+U 1 1 5811BDCB
+P 25975 15800
+F 0 "Q?" V 26300 15950 50  0000 R CNN
+F 1 "J201" V 26200 15975 50  0000 R CNN
+F 2 "MyModules:SOT23-132-JRL" H 26175 15900 29  0001 C CNN
+F 3 "" H 25975 15800 60  0000 C CNN
+	1    25975 15800
+	0    1    -1   0
+$EndComp
+$Comp
+L Q_NJFET_DSG Q?
+U 1 1 5811D0E5
+P 13750 20025
+F 0 "Q?" V 14075 20175 50  0000 R CNN
+F 1 "J201" V 13975 20200 50  0000 R CNN
+F 2 "MyModules:SOT23-132-JRL" H 13950 20125 29  0001 C CNN
+F 3 "" H 13750 20025 60  0000 C CNN
+	1    13750 20025
+	0    -1   -1   0
+$EndComp
 $EndSCHEMATC
