File: voice.sch (KiCad schematic (older format))
At the start: 177 parts, among them U10 LM13700, U11 TA75S558F, U12 CD4053, U13 CD4053, U14 LM13700, U15 LM13700, U15 TA75S558F, U16 LM13700, U17 TL072-, U18 LM13700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

Commit message: changed NPN and PNP BJTs to modern SOT-23 equivalents
Parts:
- removed Q? (x9): MMBT3906, SOT-23, symbol MMBT3906
- removed Q?: MMBT3904, SOT-23, symbol MMBT3904
- added Q? (x9): 2SA1832, SOT-23, symbol 2SA1832
- added Q?: 2SC4738, SOT-23, symbol 2SC4738
- Q?: value MMBT3906 -> 2SA1832; symbol MMBT3906 -> 2SA1832
Connections:
- net GND: now also Q?.1 (B), Q?.1 (B), Q?.1 (B), Q?.1 (B), Q?.1 (B), Q?.1 (B), Q?.1 (B), Q?.1 (B), Q?.1 (B), Q?.2 (E)
- net at R?.2: now also Q?.2 (E) (x5)
- net at U14.1: now also Q?.3 (C)
- net at U23.12: now also Q?.2 (E)
- net at U23.16: now also Q?.3 (C)
- net at R?.1: now also Q?.2 (E) (x2)
- net at U15.16: now also Q?.3 (C)
- net at U21.1: now also Q?.3 (C)
- net at U16.1: now also Q?.3 (C)
- net at R?.1, R?.2: now also Q?.2 (E)
- net at U10.16: now also Q?.3 (C)
- net at R?.1, R?.2: now also Q?.3 (C)
- net at R?.2: now also Q?.1 (B)
- net at U16.16: now also Q?.3 (C)
- net at U23.1: now also Q?.3 (C)
- net at U10.1: now also Q?.3 (C)
Changed lines of the file:
@@
 $EndComp
 $Comp
-L MMBT3906 Q?
-U 1 1 57F1A9C4
-P 17875 8625
-F 0 "Q?" H 18075 8700 50  0000 L CNN
-F 1 "MMBT3906" V 17850 8100 50  0000 L CNN
-F 2 "SOT-23" H 18075 8550 50  0001 L CIN
-F 3 "" H 17875 8625 50  0000 L CNN
-	1    17875 8625
-	0    1    -1   0
-$EndComp
-$Comp
 L +12V #PWR?
 U 1 1 57F203E2
@@
 $EndComp
 $Comp
-L MMBT3906 Q?
-U 1 1 57F5CD40
-P 4825 16325
-F 0 "Q?" H 5025 16400 50  0000 L CNN
-F 1 "MMBT3906" V 4800 15800 50  0000 L CNN
-F 2 "SOT-23" H 5025 16250 50  0001 L CIN
-F 3 "" H 4825 16325 50  0000 L CNN
-	1    4825 16325
-	0    1    -1   0
-$EndComp
-$Comp
 L R_US R?
 U 1 1 57F5CD5F
@@
 $EndComp
 $Comp
-L MMBT3906 Q?
-U 1 1 57F78950
-P 8875 14175
-F 0 "Q?" H 9075 14250 50  0000 L CNN
-F 1 "MMBT3906" V 8850 13650 50  0000 L CNN
-F 2 "SOT-23" H 9075 14100 50  0001 L CIN
-F 3 "" H 8875 14175 50  0000 L CNN
-	1    8875 14175
-	0    1    -1   0
-$EndComp
-$Comp
 L R_US R?
 U 1 1 57F78959
@@
 $EndComp
 $Comp
-L MMBT3906 Q?
-U 1 1 58016B97
-P 28975 16025
-F 0 "Q?" H 29175 16100 50  0000 L CNN
-F 1 "MMBT3906" H 28600 16250 50  0000 L CNN
-F 2 "SOT-23" H 29175 15950 50  0001 L CIN
-F 3 "" H 28975 16025 50  0000 L CNN
-	1    28975 16025
-	1    0    0    -1
-$EndComp
-$Comp
 L +12V #PWR?
 U 1 1 58016BA1
@@
 $EndComp
 $Comp
-L MMBT3906 Q?
-U 1 1 57F4F312
-P 29100 17800
-F 0 "Q?" H 29300 17875 50  0000 L CNN
-F 1 "MMBT3906" H 28725 18025 50  0000 L CNN
-F 2 "SOT-23" H 29300 17725 50  0001 L CIN
-F 3 "" H 29100 17800 50  0000 L CNN
-	1    29100 17800
-	0    -1   -1   0
-$EndComp
-$Comp
 L R_US R?
 U 1 1 57F4FF0D
@@
 $EndComp
 $Comp
-L MMBT3906 Q?
-U 1 1 57F765B6
-P 10950 20625
-F 0 "Q?" H 11150 20700 50  0000 L CNN
-F 1 "MMBT3906" V 10900 20750 50  0000 L CNN
-F 2 "SOT-23" H 11150 20550 50  0001 L CIN
-F 3 "" H 10950 20625 50  0000 L CNN
-	1    10950 20625
-	0    1    -1   0
-$EndComp
-$Comp
 L R_US R?
 U 1 1 57F765BF
@@
 $EndComp
 $Comp
-L MMBT3906 Q?
+L 2SA1832 Q?
 U 1 1 57F7F7DA
 P 9475 18525
 F 0 "Q?" H 9675 18600 50  0000 L CNN
-F 1 "MMBT3906" V 9400 18625 50  0000 L CNN
+F 1 "2SA1832" V 9400 18625 50  0000 L CNN
 F 2 "SOT-23" H 9675 18450 50  0001 L CIN
 F 3 "" H 9475 18525 50  0000 L CNN
@@
 $EndComp
 $Comp
-L MMBT3906 Q?
-U 1 1 58022650
-P 15250 4600
-F 0 "Q?" H 15450 4675 50  0000 L CNN
-F 1 "MMBT3906" V 15225 4075 50  0000 L CNN
-F 2 "SOT-23" H 15450 4525 50  0001 L CIN
-F 3 "" H 15250 4600 50  0000 L CNN
-	1    15250 4600
-	0    1    -1   0
-$EndComp
-$Comp
 L +12V #PWR?
 U 1 1 58022656
@@
 $EndComp
 $Comp
-L MMBT3906 Q?
-U 1 1 57F82873
-P 23725 4525
-F 0 "Q?" H 23925 4600 50  0000 L CNN
-F 1 "MMBT3906" V 23700 4000 50  0000 L CNN
-F 2 "SOT-23" H 23925 4450 50  0001 L CIN
-F 3 "" H 23725 4525 50  0000 L CNN
-	1    23725 4525
-	0    1    -1   0
-$EndComp
-$Comp
 L +12V #PWR?
 U 1 1 57F82879
@@
 	13000 21200 13175 21200
 $Comp
-L MMBT3904 Q?
-U 1 1 57FA763D
-P 13525 21525
-F 0 "Q?" H 13725 21600 50  0000 L CNN
-F 1 "MMBT3904" H 13725 21525 50  0000 L CNN
-F 2 "SOT-23" H 13725 21450 50  0001 L CIN
-F 3 "" H 13525 21525 50  0000 L CNN
-	1    13525 21525
-	1    0    0    -1
-$EndComp
-$Comp
 L R_US R?
 U 1 1 57FA7BA1
@@
 VCO2_LEVEL
 $Comp
-L MMBT3906 Q?
-U 1 1 5809D2EC
-P 28025 11875
-F 0 "Q?" H 28225 11950 50  0000 L CNN
-F 1 "MMBT3906" H 27650 12100 50  0000 L CNN
-F 2 "SOT-23" H 28225 11800 50  0001 L CIN
-F 3 "" H 28025 11875 50  0000 L CNN
-	1    28025 11875
-	0    -1   -1   0
-$EndComp
-$Comp
 L GND_R #PWR?
 U 1 1 5809EC98
@@
 	0    -1   -1   0
 $EndComp
+$Comp
+L 2SA1832 Q?
+U 1 1 585A21AC
+P 10950 20625
+F 0 "Q?" H 11150 20700 50  0000 L CNN
+F 1 "2SA1832" V 10875 20725 50  0000 L CNN
+F 2 "SOT-23" H 11150 20550 50  0001 L CIN
+F 3 "" H 10950 20625 50  0000 L CNN
+	1    10950 20625
+	0    1    -1   0
+$EndComp
+$Comp
+L 2SA1832 Q?
+U 1 1 585A3496
+P 4825 16325
+F 0 "Q?" H 5025 16400 50  0000 L CNN
+F 1 "2SA1832" V 4750 16425 50  0000 L CNN
+F 2 "SOT-23" H 5025 16250 50  0001 L CIN
+F 3 "" H 4825 16325 50  0000 L CNN
+	1    4825 16325
+	0    1    -1   0
+$EndComp
+$Comp
+L 2SA1832 Q?
+U 1 1 585A4D9C
+P 8875 14175
+F 0 "Q?" H 9075 14250 50  0000 L CNN
+F 1 "2SA1832" V 8800 14275 50  0000 L CNN
+F 2 "SOT-23" H 9075 14100 50  0001 L CIN
+F 3 "" H 8875 14175 50  0000 L CNN
+	1    8875 14175
+	0    1    -1   0
+$EndComp
+$Comp
+L 2SA1832 Q?
+U 1 1 585A6F9C
+P 29100 17800
+F 0 "Q?" H 29300 17875 50  0000 L CNN
+F 1 "2SA1832" V 29025 17900 50  0000 L CNN
+F 2 "SOT-23" H 29300 17725 50  0001 L CIN
+F 3 "" H 29100 17800 50  0000 L CNN
+	1    29100 17800
+	0    -1   -1   0
+$EndComp
+$Comp
+L 2SC4738 Q?
+U 1 1 585AA4E9
+P 13525 21525
+F 0 "Q?" H 13725 21600 50  0000 L CNN
+F 1 "2SC4738" H 13725 21525 50  0000 L CNN
+F 2 "SOT-23" H 13725 21450 50  0001 L CIN
+F 3 "" H 13525 21525 50  0000 L CNN
+	1    13525 21525
+	1    0    0    -1
+$EndComp
+$Comp
+L 2SA1832 Q?
+U 1 1 585ADF1E
+P 17875 8625
+F 0 "Q?" H 18075 8700 50  0000 L CNN
+F 1 "2SA1832" H 18075 8625 50  0000 L CNN
+F 2 "SOT-23" H 18075 8550 50  0001 L CIN
+F 3 "" H 17875 8625 50  0000 L CNN
+	1    17875 8625
+	0    1    -1   0
+$EndComp
+$Comp
+L 2SA1832 Q?
+U 1 1 585B18B5
+P 15250 4600
+F 0 "Q?" H 15450 4675 50  0000 L CNN
+F 1 "2SA1832" H 15450 4600 50  0000 L CNN
+F 2 "SOT-23" H 15450 4525 50  0001 L CIN
+F 3 "" H 15250 4600 50  0000 L CNN
+	1    15250 4600
+	0    1    -1   0
+$EndComp
+$Comp
+L 2SA1832 Q?
+U 1 1 585B2849
+P 23725 4525
+F 0 "Q?" H 23925 4600 50  0000 L CNN
+F 1 "2SA1832" H 23925 4525 50  0000 L CNN
+F 2 "SOT-23" H 23925 4450 50  0001 L CIN
+F 3 "" H 23725 4525 50  0000 L CNN
+	1    23725 4525
+	0    1    -1   0
+$EndComp
+$Comp
+L 2SA1832 Q?
+U 1 1 585B8A1E
+P 28975 16025
+F 0 "Q?" H 29175 16100 50  0000 L CNN
+F 1 "2SA1832" V 28900 16125 50  0000 L CNN
+F 2 "SOT-23" H 29175 15950 50  0001 L CIN
+F 3 "" H 28975 16025 50  0000 L CNN
+	1    28975 16025
+	1    0    0    -1
+$EndComp
+$Comp
+L 2SA1832 Q?
+U 1 1 585BB02B
+P 28025 11875
+F 0 "Q?" H 28225 11950 50  0000 L CNN
+F 1 "2SA1832" V 27950 11975 50  0000 L CNN
+F 2 "SOT-23" H 28225 11800 50  0001 L CIN
+F 3 "" H 28025 11875 50  0000 L CNN
+	1    28025 11875
+	0    -1   -1   0
+$EndComp

Commit message: more transistor swapping
Parts:
- removed Q?: MMBT3906, SOT-23, symbol MMBT3906
- added Q?: 2SA1832, SOT-23, symbol 2SA1832
Connections:
- net GND: now also Q?.1 (B)
- net at U15.1: now also Q?.3 (C)
- net at R?.2: now also Q?.2 (E)
Changed lines of the file:
@@
 $EndComp
 $Comp
-L MMBT3906 Q?
-U 1 1 57F5AD92
-P 4825 14150
-F 0 "Q?" H 5025 14225 50  0000 L CNN
-F 1 "MMBT3906" V 4800 13625 50  0000 L CNN
-F 2 "SOT-23" H 5025 14075 50  0001 L CIN
-F 3 "" H 4825 14150 50  0000 L CNN
-	1    4825 14150
-	0    1    -1   0
-$EndComp
-$Comp
 L +12V #PWR?
 U 1 1 57F5ADA2
@@
 	0    -1   -1   0
 $EndComp
+$Comp
+L 2SA1832 Q?
+U 1 1 585B20AD
+P 4825 14150
+F 0 "Q?" H 5025 14225 50  0000 L CNN
+F 1 "2SA1832" V 4750 14250 50  0000 L CNN
+F 2 "SOT-23" H 5025 14075 50  0001 L CIN
+F 3 "" H 4825 14150 50  0000 L CNN
+	1    4825 14150
+	0    1    -1   0
+$EndComp
 $EndSCHEMATC
