File: voice.kicad_pcb (KiCad board)
At the start: 2 copper layers, 133.3 x 50 mm, 420 parts, among them J1 DDR3-DIMM, Q1 2SA1832, Q10 2SA1832, Q11 2SA1832, Q12 2SK208-GR, Q13 2SK208-GR, Q14 2SA1832, Q15 2SA1832, Q16 2SA1618, Q17 2SA1832, Q18 2SA1832, Q19 2SK208-GR, Q2 2SA1832, Q20 2SA1832, Q21 2SC4738, Q22 2SC4738, Q23 2SC4738, Q24 2SC4207, Q25 2SA1618, Q26 2SA1618, Q27 2SC4207, Q28 2SC4738, Q29 MMBF4391LT1G, Q3 2SA1832, Q30 MMBF4391LT1G, Q31 2SC4207, Q32 2SC4207, Q33 PMBT2369, Q34 PMBT2369, Q35 2SA1832, Q36 2SA1832, Q37 PMBT2369, Q38 2SC4738, Q4 2SA1832, Q5 2SK208-GR, Q6 2SK208-GR, Q7 2SK208-GR, Q8 2SK208-GR, Q9 2SK208-GR, U1 CD4053, U10 LM13700, U11 TL072-, U12 LM13700, U13 TA75S558F, U14 LM13700, U15 RC4558, U16 TA75S558F, U17 NE555, U18 NE555, U19 TL074-, U2 LM13700, U20 CD4052, U21 CD4052, U22 TL074-, U23 TL072-, U24 TL074-, U25 TA75S558F, U26 TL072-, U27 TL074-, U3 TA75S558F, U30 CD4052, U31 CD4052, U4 CD4053, U5 LM13700, U6 TA75S558F, U7 LM13700, U8 LM13700, U9 LM13700

Commit message: placing...
Parts:
- moved R63 62.6 mm to (115.0, 42.2), turned to 270 degrees
- moved R18 62.6 mm to (120.0, 37.5), turned to 90 degrees
- moved R58 60.6 mm to (115.0, 45.2), turned to 90 degrees
- moved R24 60.5 mm to (123.2, 37.5), turned to 270 degrees
- moved R64 53.4 mm to (120.0, 50.5)
- moved R49 51.2 mm to (123.0, 50.5), turned to 180 degrees
- moved U11 50.9 mm to (135.0, 41.0), turned to 180 degrees
- moved R70 50.0 mm to (128.2, 47.0), turned to 180 degrees
- moved Q10 49.7 mm to (126.0, 49.5), turned to 270 degrees
- moved R79 47.8 mm to (132.8, 46.2)
- moved R25 21.1 mm to (121.0, 28.0), turned to 180 degrees
- moved R27 19.1 mm to (121.0, 29.8), turned to 0 degrees
- moved R19 15.9 mm to (128.2, 44.5), turned to 0 degrees
- moved R28 14.0 mm to (128.2, 42.8), turned to 180 degrees
- moved R22 13.1 mm to (130.2, 28.0), turned to 180 degrees
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Connections:
- U10 pad 1: Net-(Q10-Pad3) -> Net-(U10-Pad1)
- U10 pad 2: Net-(R49-Pad1) -> Net-(U10-Pad2)
- U10 pad 3: Net-(R64-Pad2) -> Net-(U10-Pad3)
- U10 pad 4: Net-(R58-Pad2) -> Net-(U10-Pad4)
- U10 pad 5: Net-(C4-Pad2) -> Net-(U10-Pad5)
- U5 pad 12: Net-(U5-Pad12) -> Net-(C4-Pad2)
- U5 pad 13: Net-(U5-Pad13) -> Net-(R58-Pad2)
- U5 pad 14: Net-(U5-Pad14) -> Net-(R64-Pad2)
- U5 pad 15: Net-(U5-Pad15) -> Net-(R49-Pad1)
- U5 pad 16: Net-(U5-Pad16) -> Net-(Q10-Pad3)
Routing:
- net VCO2: track 0.00 -> 9.82 mm
- net Net-(R20-Pad1): track 0.00 -> 8.23 mm
- net Net-(R29-Pad2): track 0.00 -> 6.55 mm
- net Net-(R25-Pad1): track 0.00 -> 6.43 mm
- net Net-(U4-Pad14): track 0.00 -> 5.90 mm
- net VCO2_PULSE: track 5.28 -> 0.00 mm
- net Net-(R19-Pad1): track 0.00 -> 4.94 mm
- net Net-(R32-Pad2): track 0.00 -> 4.26 mm
- net Net-(D11-Pad2): track 0.00 -> 3.78 mm
- net Net-(R21-Pad1): track 0.00 -> 2.27 mm
- net Net-(C31-Pad2): track 34.6 -> 36.1 mm
- net VCO2_AUTOTUNE: track 0.00 -> 1.40 mm
- net VCO2_SAW: track 10.7 -> 11.7 mm
