File: envelopes.sch (KiCad schematic (older format))
At the start: 77 parts, among them U25 TL074-, U26 CD4052, U27 NE555, U28 TL074-, U29 CD4052, U30 NE555

Commit message: litte bit of work again - added tri sym CVs
Changed lines of the file:
@@
 	2975 12275 2725 12275
 Wire Wire Line
-	2725 12275 2725 12625
-Wire Wire Line
-	2725 12625 2725 12975
-Wire Wire Line
-	2725 12975 2725 13275
-Wire Wire Line
-	2725 13275 2725 13475
-Wire Wire Line
-	2725 13475 2725 13725
+	2725 12275 2725 13725
 Wire Wire Line
 	2725 12625 2975 12625
@@
 	2975 12125 2525 12125
 Wire Wire Line
-	2525 11475 2525 12125
-Wire Wire Line
-	2525 12125 2525 12425
+	2525 11475 2525 12425
 Wire Wire Line
 	2525 12425 2975 12425
@@
 	9975 12200 9575 12200
 Wire Wire Line
-	9575 12200 9575 13075
-Wire Wire Line
-	9575 13075 9575 13675
+	9575 12200 9575 13675
 Wire Wire Line
 	10575 12975 10675 12975
 Wire Wire Line
-	10575 13175 10625 13175
-Wire Wire Line
-	10625 13175 10675 13175
+	10575 13175 10675 13175
 Wire Wire Line
 	10625 13175 10625 13825
@@
 	9575 13675 9125 13675
 Wire Wire Line
-	9425 11875 9425 11925
-Wire Wire Line
-	9425 11925 9425 12700
+	9425 11875 9425 12700
 Wire Wire Line
 	9425 12700 9325 12700
@@
 	8575 11925 8025 11925
 Wire Wire Line
-	8025 10925 8025 11925
-Wire Wire Line
-	8025 11925 8025 12600
-Wire Wire Line
-	8025 12600 8025 13675
+	8025 10925 8025 13675
 Wire Wire Line
 	8025 12600 8325 12600
@@
 	11625 12975 11075 12975
 Wire Wire Line
-	26600 11125 26750 11125
-Wire Wire Line
-	26750 11125 27400 11125
+	26600 11125 27400 11125
 Connection ~ 11625 11125
 Wire Wire Line
@@
 	8025 13675 8725 13675
 Wire Wire Line
-	2175 9525 2525 9525
-Wire Wire Line
-	2525 9525 2575 9525
-Wire Wire Line
-	2975 9525 3125 9525
-Wire Wire Line
-	3125 9525 3275 9525
+	2175 9525 2575 9525
+Wire Wire Line
+	2975 9525 3275 9525
 Wire Wire Line
 	2525 10125 2525 10325
@@
 	3575 9925 3575 9725
 Wire Wire Line
-	4275 9125 4475 9125
-Wire Wire Line
-	4475 9125 4925 9125
-Wire Wire Line
-	3575 9125 3725 9125
-Wire Wire Line
-	3725 9125 3875 9125
-Wire Wire Line
-	3575 9025 3575 9125
-Wire Wire Line
-	3575 9125 3575 9325
+	4275 9125 4925 9125
+Wire Wire Line
+	3575 9125 3875 9125
+Wire Wire Line
+	3575 9025 3575 9325
 Connection ~ 3575 9125
 Wire Wire Line
@@
 	4875 9775 4875 10325
 Wire Wire Line
-	6325 9775 6425 9775
-Wire Wire Line
-	6425 9775 6475 9775
+	6325 9775 6475 9775
 Wire Wire Line
 	6475 8575 6475 9775
 Wire Wire Line
-	3575 8575 4475 8575
-Wire Wire Line
-	4475 8575 4675 8575
-Wire Wire Line
-	4675 8575 5075 8575
-Wire Wire Line
-	5075 8575 6475 8575
+	3575 8575 6475 8575
 Wire Wire Line
 	3575 8575 3575 8625
@@
 	2200 10975 4625 10975
 Wire Wire Line
-	7525 10125 7525 10975
-Wire Wire Line
-	7525 10975 7525 11125
+	7525 10125 7525 11125
 Connection ~ 7525 10975
 Wire Wire Line
-	9325 10825 9425 10825
-Wire Wire Line
-	9425 10825 9525 10825
-Wire Wire Line
-	9325 11025 9425 11025
-Wire Wire Line
-	9425 11025 9525 11025
+	9325 10825 9525 10825
+Wire Wire Line
+	9325 11025 9525 11025
 Connection ~ 9425 11025
 Connection ~ 9425 10825
 Wire Wire Line
-	8525 10825 8525 10925
-Wire Wire Line
-	8525 10925 8525 11025
+	8525 10825 8525 11025
 Wire Wire Line
 	9125 11325 9125 11425
@@
 	9725 11325 9725 11425
 Wire Wire Line
-	9925 10825 10400 10825
-Wire Wire Line
-	10400 10825 10575 10825
-Wire Wire Line
-	9925 11025 10400 11025
-Wire Wire Line
-	10400 11025 10475 11025
+	9925 10825 10575 10825
+Wire Wire Line
+	9925 11025 10475 11025
 Wire Wire Line
 	8025 10925 8525 10925
@@
 	5025 10975 5375 10975
 Wire Wire Line
-	5775 10975 7175 10975
-Wire Wire Line
-	7175 10975 7525 10975
+	5775 10975 7525 10975
 Wire Wire Line
 	5125 12375 5325 12375
 Connection ~ 7175 10975
 Wire Wire Line
-	5725 12375 5925 12375
-Wire Wire Line
-	5925 12375 6625 12375
-Wire Wire Line
-	6625 12375 6825 12375
+	5725 12375 6825 12375
 Connection ~ 5925 12375
 Connection ~ 6625 12375
@@
 	18100 12275 17850 12275
 Wire Wire Line
-	17850 12275 17850 12625
-Wire Wire Line
-	17850 12625 17850 12975
-Wire Wire Line
-	17850 12975 17850 13275
-Wire Wire Line
-	17850 13275 17850 13475
-Wire Wire Line
-	17850 13475 17850 13725
+	17850 12275 17850 13725
 Wire Wire Line
 	17850 12625 18100 12625
@@
 	18100 12125 17650 12125
 Wire Wire Line
-	17650 11475 17650 12125
-Wire Wire Line
-	17650 12125 17650 12425
+	17650 11475 17650 12425
 Wire Wire Line
 	17650 12425 18100 12425
@@
 	25700 13600 25800 13600
 Wire Wire Line
-	25700 13800 25750 13800
-Wire Wire Line
-	25750 13800 25800 13800
+	25700 13800 25800 13800
 Wire Wire Line
 	25750 13800 25750 14200
@@
 	24700 13700 24250 13700
 Wire Wire Line
-	24550 11875 24550 11925
-Wire Wire Line
-	24550 11925 24550 12650
+	24550 11875 24550 12650
 Wire Wire Line
 	24550 12650 24450 12650
@@
 	23700 11925 23150 11925
 Wire Wire Line
-	23150 10925 23150 11925
-Wire Wire Line
-	23150 11925 23150 12550
-Wire Wire Line
-	23150 12550 23150 13700
+	23150 10925 23150 13700
 Wire Wire Line
 	23150 12550 23450 12550
@@
 	26750 13600 26200 13600
 Wire Wire Line
-	11475 11125 11625 11125
-Wire Wire Line
-	11625 11125 11875 11125
+	11475 11125 11875 11125
 Connection ~ 26750 11125
 Wire Wire Line
@@
 	23150 13700 23850 13700
 Wire Wire Line
-	17300 9525 17650 9525
-Wire Wire Line
-	17650 9525 17700 9525
-Wire Wire Line
-	18100 9525 18250 9525
-Wire Wire Line
-	18250 9525 18400 9525
+	17300 9525 17700 9525
+Wire Wire Line
+	18100 9525 18400 9525
 Wire Wire Line
 	17650 10125 17650 10325
@@
 	18700 9925 18700 9725
 Wire Wire Line
-	19400 9125 19600 9125
-Wire Wire Line
-	19600 9125 20050 9125
-Wire Wire Line
-	18700 9125 18850 9125
-Wire Wire Line
-	18850 9125 19000 9125
-Wire Wire Line
-	18700 9025 18700 9125
-Wire Wire Line
-	18700 9125 18700 9325
+	19400 9125 20050 9125
+Wire Wire Line
+	18700 9125 19000 9125
+Wire Wire Line
+	18700 9025 18700 9325
 Connection ~ 18700 9125
 Wire Wire Line
@@
 	20000 9775 20000 10325
 Wire Wire Line
-	21450 9775 21550 9775
-Wire Wire Line
-	21550 9775 21600 9775
+	21450 9775 21600 9775
 Wire Wire Line
 	21600 8575 21600 9775
 Wire Wire Line
-	18700 8575 19600 8575
-Wire Wire Line
-	19600 8575 19800 8575
-Wire Wire Line
-	19800 8575 20200 8575
-Wire Wire Line
-	20200 8575 21600 8575
+	18700 8575 21600 8575
 Wire Wire Line
 	18700 8575 18700 8625
@@
 	17350 10975 19750 10975
 Wire Wire Line
-	22650 10125 22650 10975
-Wire Wire Line
-	22650 10975 22650 11125
+	22650 10125 22650 11125
 Connection ~ 22650 10975
 Wire Wire Line
-	23650 10825 23650 10925
-Wire Wire Line
-	23650 10925 23650 11025
+	23650 10825 23650 11025
 Wire Wire Line
 	24250 11325 24250 11425
@@
 	24850 11325 24850 11425
 Wire Wire Line
-	25050 10825 25525 10825
-Wire Wire Line
-	25525 10825 25700 10825
-Wire Wire Line
-	25050 11025 25525 11025
-Wire Wire Line
-	25525 11025 25600 11025
+	25050 10825 25700 10825
+Wire Wire Line
+	25050 11025 25600 11025
 Wire Wire Line
 	23150 10925 23650 10925
@@
 	20150 10975 20500 10975
 Wire Wire Line
-	20900 10975 22300 10975
-Wire Wire Line
-	22300 10975 22650 10975
+	20900 10975 22650 10975
 Wire Wire Line
 	20250 12375 20450 12375
 Connection ~ 22300 10975
 Wire Wire Line
-	20850 12375 21050 12375
-Wire Wire Line
-	21050 12375 21750 12375
-Wire Wire Line
-	21750 12375 21950 12375
+	20850 12375 21950 12375
 Connection ~ 21050 12375
 Connection ~ 21750 12375
@@
 	21450 9575 26750 9575
 Wire Wire Line
-	26750 9575 26750 10575
-Wire Wire Line
-	26750 10575 26750 11125
-Wire Wire Line
-	26750 11125 26750 13600
+	26750 9575 26750 13600
 Wire Wire Line
 	21050 12375 21050 12675
@@
 	27400 10300 28475 10300
 Wire Wire Line
-	28400 11025 28475 11025
-Wire Wire Line
-	28475 11025 28600 11025
+	28400 11025 28600 11025
 Wire Wire Line
 	28475 10300 28475 11025
@@
 ENV_1
 Wire Wire Line
-	13825 11025 13900 11025
-Wire Wire Line
-	13900 11025 14025 11025
+	13825 11025 14025 11025
 Connection ~ 13900 11025
 $Comp
@@
 	12700 10375 12700 10925
 Wire Wire Line
-	12425 10925 12700 10925
-Wire Wire Line
-	12700 10925 12825 10925
+	12425 10925 12825 10925
 $Comp
 L R_US R?
@@
 $EndComp
 Wire Wire Line
-	12275 11125 12325 11125
-Wire Wire Line
-	12325 11125 12375 11125
+	12275 11125 12375 11125
 Wire Wire Line
 	12325 11125 12325 11400
@@
 	11625 9000 11625 9075
 Wire Wire Line
-	11625 9575 11625 10575
-Wire Wire Line
-	11625 10575 11625 10925
-Wire Wire Line
-	11625 10925 11625 11125
-Wire Wire Line
-	11625 11125 11625 12975
+	11625 9575 11625 12975
 NoConn ~ 11625 9475
 Text Notes 11675 9450 0    50   ~ 0
@@
 	8525 11025 8925 11025
 Wire Wire Line
-	9425 10825 9425 11025
-Wire Wire Line
-	9425 11025 9425 11475
-Wire Wire Line
-	24450 10825 24550 10825
-Wire Wire Line
-	24550 10825 24650 10825
-Wire Wire Line
-	24450 11025 24550 11025
-Wire Wire Line
-	24550 11025 24650 11025
+	9425 10825 9425 11475
+Wire Wire Line
+	24450 10825 24650 10825
+Wire Wire Line
+	24450 11025 24650 11025
 Connection ~ 24550 11025
 Connection ~ 24550 10825
@@
 $EndComp
 Wire Wire Line
-	24550 10825 24550 11025
-Wire Wire Line
-	24550 11025 24550 11475
+	24550 10825 24550 11475
 Wire Wire Line
 	24050 10825 23650 10825

Commit message: more voice work
Changed lines of the file:
@@
 	6325 9775 6475 9775
 Wire Wire Line
-	6475 8575 6475 9775
-Wire Wire Line
-	3575 8575 6475 8575
+	6475 9775 6475 8575
+Wire Wire Line
+	6475 8575 3575 8575
 Wire Wire Line
 	3575 8575 3575 8625
@@
 	21450 9775 21600 9775
 Wire Wire Line
-	21600 8575 21600 9775
-Wire Wire Line
-	18700 8575 21600 8575
+	21600 9775 21600 8575
+Wire Wire Line
+	21600 8575 18700 8575
 Wire Wire Line
 	18700 8575 18700 8625

Commit message: annotated, added decoupling caps
Parts:
- removed Q? (x4): PMP4201G, TO_SOT_Packages_SMD:SOT-353_SC-70-5, symbol PMP4201G
- removed Q? (x4): PMP5201G, TO_SOT_Packages_SMD:SOT-353_SC-70-5, symbol PMP5201G
- added Q24, Q27: 2SC4207, TO_SOT_Packages_SMD:SOT-353_SC-70-5, symbol 2SC4207
- added Q25, Q26: 2SA1618, TO_SOT_Packages_SMD:SOT-353_SC-70-5, symbol 2SA1618
- gave numbers to parts that had none: 63
- renumbered U27 to U17, U30 to U18, U25 to U19, U26 to U20, U29 to U21, U28 to U22
Connections:
- net ENV_2: now also U22.8, U22.9 (-); no longer U22.13 (-), U22.14
- net GND: now also Q24.3 (B), Q25.3 (B), Q26.3 (B), Q27.3 (B)
- net at C25.2, R162.1, U19.2 (-): now also Q24.5 (C), Q25.4 (C)
- net at C24.1, R161.2, U18.6 (THR)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: now also U22.10 (+); no longer U22.12 (+)
- net at R145.2: now also Q24.2 (E), Q24.2 (E), Q25.2 (E), Q25.2 (E)
- net at C23.2, U19.6 (-): now also Q24.4 (C), Q25.5 (C)
- net at R149.2, R152.2, R153.2: now also Q25.1 (B)
- net at R135.2, R140.2, R141.2: now also Q24.1 (B)
- net at C26.2, R163.1, U22.2 (-): now also Q26.4 (C), Q27.5 (C)
- net at R164.1, R166.2: now also U22.12 (+); no longer U22.5 (+)
- net at R160.2, R161.1: now also U22.13 (-); no longer U22.6 (-)
- net at R160.1, R163.2: now also U22.14; no longer U22.7
- net at R146.2: now also Q26.2 (E), Q26.2 (E), Q27.2 (E), Q27.2 (E)
- net at C24.2, U22.6 (-): now also Q26.5 (C), Q27.4 (C)
- net at R151.2, R154.2, R155.2: now also Q26.1 (B)
- net at R137.2, R142.2, R143.2: now also Q27.1 (B)

Commit message: starting placing VCO1
Parts:
- Q22, Q23, Q28: footprint SOT-23 -> MyModules:SOT416-SC75
Changed lines of the file:
@@
 F 0 "Q28" H 12625 11675 50  0000 L CNN
 F 1 "2SC4738" H 12625 11600 50  0000 L CNN
-F 2 "SOT-23" H 12625 11525 50  0001 L CIN
+F 2 "MyModules:SOT416-SC75" H 12625 11525 50  0001 L CIN
 F 3 "" H 12425 11600 50  0000 L CNN
 	1    12425 11600
@@
 F 0 "Q23" H 18250 9750 50  0000 L CNN
 F 1 "2SC4738" H 18250 9675 50  0000 L CNN
-F 2 "SOT-23" H 18800 9450 50  0001 L CIN
+F 2 "MyModules:SOT416-SC75" H 18800 9450 50  0001 L CIN
 F 3 "" H 18600 9525 50  0000 L CNN
 	1    18600 9525
@@
 F 0 "Q22" H 3075 9750 50  0000 L CNN
 F 1 "2SC4738" H 3075 9675 50  0000 L CNN
-F 2 "SOT-23" H 3675 9450 50  0001 L CIN
+F 2 "MyModules:SOT416-SC75" H 3675 9450 50  0001 L CIN
 F 3 "" H 3475 9525 50  0000 L CNN
 	1    3475 9525
